Commit message: add ros2 controllers

File: fiar_pkg/urdf/fiarURDF.urdf.xacro (robot description, xacro)
@@ -25,47 +25,47 @@
     </link>
     <!-- ========= Xacro Include Legs=========-->
-    <xacro:front_leg link1="legR1" link2="legR2" wheel="wR1" joint1="legR2_to_legR1" joint2="wheel_to_legR2" />
-    <xacro:front_leg link1="legL1" link2="legL2" wheel="wL1" joint1="legL2_to_legL1" joint2="wheel_to_legL2"/>
-    <xacro:front_leg link1="legBackR1" link2="legBackR2" wheel="wR2" joint1="legBackR2_to_legBackR1" joint2="wheel_to_legBackR2"/>
-    <xacro:front_leg link1="legBackL1" link2="legBackL2" wheel="wL2" joint1="legBackL2_to_legBackL1" joint2="wheel_to_legBackL2"/>
+    <xacro:front_leg link1="legR1" link2="legR2" wheel="wR1" joint1="LF2" joint2="w1" />
+    <xacro:front_leg link1="legL1" link2="legL2" wheel="wL1" joint1="RF2" joint2="w2"/>
+    <xacro:front_leg link1="legBackR1" link2="legBackR2" wheel="wR2" joint1="RB2" joint2="w3"/>
+    <xacro:front_leg link1="legBackL1" link2="legBackL2" wheel="wL2" joint1="LB2" joint2="w4"/>
     <!-- === Xacro Include Head ====-->
     <xacro:topHead head="head" neck="neck"/>
     <!-- === leg1_to_body ===-->
-    <joint name="legL1_to_body" type="revolute">
+    <joint name="LF1" type="revolute">
         <parent link="body"/>
         <child link="legR1"/>
         <origin xyz="0.125 0.1 0" rpy="1.5707 0 0"/>
         <axis xyz="0 0 1"/>
-        <limit lower="-0" upper="-3.1415" effort="0.01" velocity="0.4"/>
+        <limit lower="-3.1415" upper="0" effort="10" velocity="0.4"/>
         <dynamics damping="1" friction="1"/>
     </joint>
     <!-- === leg2_to_body ===-->
-    <joint name="legL2_to_body" type="revolute">
+    <joint name="RF1" type="revolute">
         <parent link="body"/>
         <child link="legL1"/>
         <origin xyz="0.125 -0.1 0" rpy="-1.5707 0 0"/>
         <axis xyz="0 0 -1"/>
-        <limit lower="0" upper="-3.1415" effort="0.01" velocity="0.4"/>
+        <limit lower="-3.1415" upper="0" effort="10" velocity="0.4"/>
         <dynamics damping="1" friction="1"/>
     </joint>
     <!-- === leg3_to_body === -->
-    <joint name="legB1_to_body" type="revolute">
+    <joint name="LB1" type="revolute">
         <parent link="body"/>
         <child link="legBackR1"/>
         <origin xyz="-0.125 0.1 0" rpy="1.5707 0 0"/>
         <axis xyz="0 0 1"/>
-        <limit lower="0" upper="-3.1415" effort="0.01" velocity="0.4"/>
+        <limit lower="-3.1415" upper="0" effort="10" velocity="0.4"/>
         <dynamics damping="1" friction="1"/>
     </joint>
     <!-- === leg4_to_body ===-->
-    <joint name="legB2_to_body" type="revolute">
+    <joint name="RB1" type="revolute">
         <parent link="body"/>
         <child link="legBackL1"/>
         <origin xyz="-0.125 -0.1 0" rpy="-1.5707 0 0"/>
         <axis xyz="0 0 -1"/>
-        <limit lower="0" upper="-3.1415" effort="0.01" velocity="0.4"/>
+        <limit lower="-3.1415" upper="0" effort="10" velocity="0.4"/>
          <dynamics damping="1" friction="1"/>
     </joint>
-    <!-- === Head to Boty ===-->
+    <!-- === Head to Body ===-->
     <joint name="neck_to_body" type="revolute">
         <parent link="body"/>
@@ -73,6 +73,8 @@
         <origin xyz="0.14 0 0.0875"/>
         <axis xyz="0 0 1"/>
-        <limit lower="0" upper="-3.1415" effort="0.01" velocity="0.4"/>
+        <limit lower="-3.1415" upper="0" effort="10" velocity="0.4"/>
          <dynamics damping="1" friction="1"/>
     </joint>
+<!-- Control interface -->
+  <xacro:include filename="$(find fiar_pkg)/urdf/controls.urdf.xacro"/>
 </robot>

File: fiar_pkg/urdf/frontLeg.urdf.xacro (robot description, xacro)
@@ -75,5 +75,5 @@
             <origin xyz="0.10 0 0.03"/>
             <axis xyz="0 0 1"/>
-            <limit lower="-2" upper="2" effort="0.01" velocity="0.4"/>
+            <limit lower="-2" upper="2" effort="10" velocity="0.4"/>
             <dynamics damping="1" friction="1"/>
      </joint>
@@ -132,7 +132,7 @@
         <parent link="${neck}"/>
         <child link="${head}"/>
-        <origin xyz="0 0 0.155" rpy="0 1.57 0"/>
+        <origin xyz="0 0 0.095" rpy="0 1.57 0"/>
         <axis xyz="0 0 1"/>
-        <limit lower="0" upper="-3.1415" effort="0.01" velocity="0.4"/>
+        <limit lower="-3.1415" upper="0" effort="10" velocity="0.4"/>
          <dynamics damping="1" friction="1"/>
     </joint>

Commit message: add initial pose

File: fiar_pkg/urdf/fiarURDF.urdf.xacro (robot description, xacro)
@@ -25,6 +25,6 @@
     </link>
     <!-- ========= Xacro Include Legs=========-->
-    <xacro:front_leg link1="legR1" link2="legR2" wheel="wR1" joint1="LF2" joint2="w1" />
-    <xacro:front_leg link1="legL1" link2="legL2" wheel="wL1" joint1="RF2" joint2="w2"/>
+    <xacro:front_leg link1="legL1" link2="legL2" wheel="wL1" joint1="LF2" joint2="w1" />
+    <xacro:front_leg link1="legR1" link2="legR2" wheel="wR1" joint1="RF2" joint2="w2"/>
     <xacro:front_leg link1="legBackR1" link2="legBackR2" wheel="wR2" joint1="RB2" joint2="w3"/>
     <xacro:front_leg link1="legBackL1" link2="legBackL2" wheel="wL2" joint1="LB2" joint2="w4"/>
@@ -34,8 +34,8 @@
     <joint name="LF1" type="revolute">
         <parent link="body"/>
-        <child link="legR1"/>
+        <child link="legL1"/>
         <origin xyz="0.125 0.1 0" rpy="1.5707 0 0"/>
         <axis xyz="0 0 1"/>
-        <limit lower="-3.1415" upper="0" effort="10" velocity="0.4"/>
+        <limit lower="-3.1415" upper="0" effort="10" velocity="2"/>
         <dynamics damping="1" friction="1"/>
     </joint>
@@ -43,26 +43,26 @@
     <joint name="RF1" type="revolute">
         <parent link="body"/>
-        <child link="legL1"/>
+        <child link="legR1"/>
         <origin xyz="0.125 -0.1 0" rpy="-1.5707 0 0"/>
         <axis xyz="0 0 -1"/>
-        <limit lower="-3.1415" upper="0" effort="10" velocity="0.4"/>
+        <limit lower="-3.1415" upper="0" effort="10" velocity="2"/>
         <dynamics damping="1" friction="1"/>
     </joint>
     <!-- === leg3_to_body === -->
-    <joint name="LB1" type="revolute">
+    <joint name="RB1" type="revolute">
         <parent link="body"/>
         <child link="legBackR1"/>
         <origin xyz="-0.125 0.1 0" rpy="1.5707 0 0"/>
         <axis xyz="0 0 1"/>
-        <limit lower="-3.1415" upper="0" effort="10" velocity="0.4"/>
+        <limit lower="-3.1415" upper="0" effort="10" velocity="2"/>
         <dynamics damping="1" friction="1"/>
     </joint>
     <!-- === leg4_to_body ===-->
-    <joint name="RB1" type="revolute">
+    <joint name="LB1" type="revolute">
         <parent link="body"/>
         <child link="legBackL1"/>
         <origin xyz="-0.125 -0.1 0" rpy="-1.5707 0 0"/>
         <axis xyz="0 0 -1"/>
-        <limit lower="-3.1415" upper="0" effort="10" velocity="0.4"/>
+        <limit lower="-3.1415" upper="0" effort="10" velocity="2"/>
          <dynamics damping="1" friction="1"/>
     </joint>
@@ -73,5 +73,5 @@
         <origin xyz="0.14 0 0.0875"/>
         <axis xyz="0 0 1"/>
-        <limit lower="-3.1415" upper="0" effort="10" velocity="0.4"/>
+        <limit lower="-3.1415" upper="0" effort="10" velocity="2"/>
          <dynamics damping="1" friction="1"/>
     </joint>
