Commit message: separate head controllers from the 'fiar_controllers'

File: fiar_pkg/urdf/controls.urdf.xacro (robot description, xacro)
@@ -113,12 +113,12 @@
         <plugin filename="gz_ros2_control-system" name="gz_ros2_control::GazeboSimROS2ControlPlugin">
             <parameters>$(find  fiar_pkg)/config/gz_parameters.yaml</parameters>
-            <position_proportional_gain>10.0</position_proportional_gain>
+            <!-- <position_proportional_gain>10.0</position_proportional_gain>
             <position_integral_gain>0.0</position_integral_gain>
             <position_derivative_gain>1.0</position_derivative_gain>
             <velocity_proportional_gain>10.0</velocity_proportional_gain>
             <velocity_integral_gain>0.0</velocity_integral_gain>
-            <velocity_derivative_gain>1.0</velocity_derivative_gain>
+            <velocity_derivative_gain>1.0</velocity_derivative_gain> -->
         </plugin>
     </gazebo>
-    <!-- <xacro:include filename="$(find  fiar_pkg)/urdf/pid_control_joint_position.urdf.xacro"/> -->
+    <xacro:include filename="$(find  fiar_pkg)/urdf/pid_control_joint_position.urdf.xacro"/>
 </robot>

File: fiar_pkg/urdf/fiarURDF.urdf.xacro (robot description, xacro)
@@ -45,12 +45,12 @@
         <child link="legR1"/>
         <origin xyz="0.125 -0.1 0" rpy="-1.5707 0 0"/>
-        <axis xyz="0 0 -1"/>
-        <limit lower="-3.1415" upper="0" effort="10" velocity="2"/>
+        <axis xyz="0 0 1"/>
+        <limit lower="0" upper="3.1415" effort="10" velocity="2"/>
         <dynamics damping="1" friction="1"/>
     </joint>
     <!-- === leg3_to_body === -->
-    <joint name="RB1" type="revolute">
+    <joint name="LB1" type="revolute">
         <parent link="body"/>
-        <child link="legBackR1"/>
+        <child link="legBackL1"/>
         <origin xyz="-0.125 0.1 0" rpy="1.5707 0 0"/>
         <axis xyz="0 0 1"/>
@@ -59,10 +59,10 @@
     </joint>
     <!-- === leg4_to_body ===-->
-    <joint name="LB1" type="revolute">
+    <joint name="RB1" type="revolute">
         <parent link="body"/>
-        <child link="legBackL1"/>
+        <child link="legBackR1"/>
         <origin xyz="-0.125 -0.1 0" rpy="-1.5707 0 0"/>
-        <axis xyz="0 0 -1"/>
-        <limit lower="-3.1415" upper="0" effort="10" velocity="2"/>
+        <axis xyz="0 0 1"/>
+        <limit lower="0" upper="3.1415" effort="10" velocity="2"/>
          <dynamics damping="1" friction="1"/>
     </joint>

File: fiar_pkg/urdf/frontLeg.urdf.xacro (robot description, xacro)
@@ -75,5 +75,5 @@
             <origin xyz="0.10 0 0.03"/>
             <axis xyz="0 0 1"/>
-            <limit lower="-2" upper="2" effort="10" velocity="0.4"/>
+            <limit lower="-2" upper="2" effort="10" velocity="1"/>
             <dynamics damping="1" friction="1"/>
      </joint>
